File: electronics/NixiePM.kicad_pcb (KiCad board)
At the start: 4 copper layers, 405 x 190 mm, 156 parts, among them J1 IN, J2 SW, J3 OUT1, J4 OUT2, U1 XSD366-094, U10 250pF 500V 5%, U11 500pF 500V 5%, U12 500pF 500V 5%, U13 500pF 500V 5%, U14 22n 630V 5%, U15 22n 630V 5%, U16 500pF 500V 5%, U17 22n 630V 5%, U18 470R 500V 2W, U19 100n 630V 5%, U2 L7812CV-DG, U20 CF2WS-82KΩ±5%_T, U21 100pF 500V 5%, U22 CR1/2W-220K±5%-XT52, U23 100n 630V 5%, U24 4n7 630V 5%, U25 22n 630V 5%, U26 22n 630V 5%, U27 CR1/2W-220K±5%-XT52, U28 CR1/2W-220K±5%-XT52, U29 CR-L5W-1KΩJ, U3 AB24S, U30 CR-L5W-1KΩJ, U31 16A 20mm 500V 5mm Plugin Fuse, U32 CR2W-4K7±5%-9T73, U33 3314G-1-503E, U34 ST-0-102-C03-N003-RS, U35 MT-0-103-C004-N004-RS, U4 CR1/2W-220K±5%-XT52, U5 CR2W-68K±5%-9T73, U6 500pF 500V 5%, U7 4n7 630V 5%, U8 2n2 630V 5%, U9 500pF 500V 5%, X12 GND_OT, X9 Audio IN

Commit message: schematic ready, layout started
Parts:
- removed AC-IN1, AC-IN2, AC-IN3, AC-IN4, AC-IN5, Audio-A1, Audio-B1, Audio-To-FX1, Audo-From-FX1, GND-AUD1, HV-B1, HV-OT1, HV-OT2, THUMP1, THUMP2: 1, TestPoint:TestPoint_THTPad_D3.0mm_Drill1.5mm
- removed AC-IN6, AC-IN7, AC-IN8: 1, TestPoint:TestPoint_THTPad_D4.0mm_Drill2.0mm
- removed AIR1, AIR10, AIR11, AIR12, AIR13, AIR14, AIR15, AIR16, AIR2, AIR3, AIR4, AIR5, AIR6, AIR7, AIR8, AIR9: VentingHole, MountingHole:MountingHole_4.3mm_M4
- removed BiasA1, BiasB1, GND-Mess1: 1, TestPoint:TestPoint_Pad_D2.0mm
- removed C10, C8, C9: 33uF 500V 5R5-ESR, footprints:CAP-TH_BD12.5-P5.00-D0.6-FD
- removed C11, C12: 18uF 450V ±20%, footprints:CAP-TH_BD10.0-P5.00-D1.0-FD
- removed C13, C14: 10uf/100V, footprints:CAP-TH_BD6.3-P2.50-D1.0-FD
- removed Choke1, Choke2: 1, TestPoint:TestPoint_THTPad_D2.5mm_Drill1.2mm
- removed D2, D5, D6: UF4007_C960666, footprints:DO-41_BD2.4-L4.7-P8.70-D0.9-RD
- removed J1: IN, wb50_footprints:WB50_Jack_TRS_6pin_16.2mm
- removed J2: SW, wb50_footprints:WB50_Jack_TRS_6pin_16.2mm
- removed J3: OUT1, wb50_footprints:WB50_Jack_TRS_6pin_16.2mm
- removed J4: OUT2, wb50_footprints:WB50_Jack_TRS_6pin_16.2mm
- removed MH3, MH4, MH5, MH6, MH7, MH8: MountHole, MountingHole:MountingHole_3.5mm_Pad_TopBottom
- removed N1, N2: ~, wb50_footprints:NetTie_0.5mm_2Pad
- removed R22, R23: CFR-25JT-52-1K5, footprints:RES-TH_BD2.4-L6.3-P10.30-D0.6
- removed R24: MOF5WS-47Ω±5%, footprints:RES-TH_BD6.0-L17.5-P21.50-D0.8
- removed R25, R26, R27: CF3WS-10KΩ±5%_T, footprints:RES-TH_BD5.5-L15.0-P19.00-D0.8
- removed R28: CR1/4W-47K±5%-ST52, footprints:RES-TH_BD2.7-L6.2-P10.20-D0.4
- removed R29: CR1/4W-15K±5%-OT52, footprints:RES-TH_BD2.7-L6.2-P10.20-D0.4
- removed R30, R31: MF1/4W-1Ω±1%-ST26, footprints:RES-TH_BD2.7-L6.2-P10.20-D0.4
- removed R32, U28: CR1/2W-220K±5%-XT52, footprints:RES-TH_BD3.5-L9.0-P13.00-D0.5
- removed RELAY1, RELAY2, RELAY3: G5V-1-12V, footprints:RELAY-TH_G5V-1
- removed RV1: Presence, wb50_footprints:WB50_Pot_Omeg_PC20BU_P5.00mm
- removed RV2: Bass, wb50_footprints:WB50_Pot_Omeg_PC20BU_P5.00mm
- removed RV3: Mid, wb50_footprints:WB50_Pot_Omeg_PC20BU_P5.00mm
- removed RV4: Treble, wb50_footprints:WB50_Pot_Omeg_PC20BU_P5.00mm
- removed RV5: Vol1, wb50_footprints:WB50_Pot_Omeg_PC20BU_P5.00mm
- removed RV6: Vol2, wb50_footprints:WB50_Pot_Omeg_PC20BU_P5.00mm
- removed RV7: Gain1, wb50_footprints:WB50_Pot_Omeg_PC20BU_P5.00mm
- removed RV8: Gain2, wb50_footprints:WB50_Pot_Omeg_PC20BU_P5.00mm
- removed U29, U30: CR-L5W-1KΩJ, footprints:RES-TH_BD9.5-L22.0-P26.00-D0.7
- removed U31: 16A 20mm 500V 5mm Plugin Fuse, footprints:FUSE-TH_L22.5-W10.8-P22.50_0031.8201.G
- removed U32: CR2W-4K7±5%-9T73, footprints:RES-TH_BD5.0-L15.5-P19.50-D0.7
- removed U33: 3314G-1-503E, footprints:RES-ADJ-SMD_3314G-1-103E
- removed U34: ST-0-102-C03-N003-RS, footprints:SW-TH_ST-0-102-C03-N003-RS
- removed U35: MT-0-103-C004-N004-RS, footprints:SW-TH_MT-0-102-C004-N004-RS
- removed V1, V2, V3: 12AX7, wb50_footprints:WB50_Socket_Noval_9Pin_D21.0mm_Hole1.8mm
- removed V4, V5: EL34, wb50_footprints:WB50_Socket_Octal_8Pin_D26.0mm_Hole2.0mm
- removed X12: GND_OT, TestPoint:TestPoint_THTPad_D4.0mm_Drill2.0mm
- removed X9: Audio IN, TestPoint:TestPoint_THTPad_D4.0mm_Drill2.0mm
- added AC1: AC ~ 230V, TestPoint:TestPoint_THTPad_D3.0mm_Drill1.5mm, F.Cu at (225.5, 69.5)
- added AC2: AC ~ 230V, TestPoint:TestPoint_THTPad_D3.0mm_Drill1.5mm, F.Cu at (225.5, 76.5)
- added NX1: IN-8, footprints:IN-8_NIXIE, F.Cu at (245.0, 234.5)
- added NX2: IN-8, footprints:IN-8_NIXIE, F.Cu at (266.0, 234.5)
- C1: value 33uF 50V -> CL10A475KO8NNNC; footprint footprints:CAP-TH_BD5.0-P2.00-D0.8-FD -> footprints:C0603
- C2: value LKMI2501C682MF -> 100nF 50V X7R; footprint footprints:CAP-TH_BD16.0-P7.50-D1.2-FD -> footprints:C0805
- C3, C4: value CC0805KRX7R9BB104 -> 100nF 50V X7R
- C5: value 0,82uF 400V 20 % -> 100nF 50V X7R; footprint footprints:CAP-TH_BD6.3-P2.50-D1.0-FD -> footprints:C0805
- C6: value 0,82uF 400V 20 % -> 33uF 500V 5R5-ESR; footprint footprints:CAP-TH_BD6.3-P2.50-D1.0-FD -> footprints:CAP-TH_BD12.5-P5.00-D0.6-FD
- C7: value 22uF_450V_16*20 -> 450BXW47MEFR16X25
- D1: value UF4007_C960666 -> MB26S_C475740; footprint footprints:DO-41_BD2.4-L4.7-P8.70-D0.9-RD -> footprints:MBS_L4.7-W4.0-P2.50-LS7.0-BL
- D3, D4: value UF4007_C960666 -> 2EZ91D5; footprint footprints:DO-41_BD2.4-L4.7-P8.70-D0.9-RD -> footprints:DO-41_BD2.4-L4.7-P8.70-D0.8-RD
- R1, R15, R6: value 33k 500V 2W -> FRC0603F6340TS; footprint footprints:RES-TH_BD3.0-L9.5-P13.50-D0.6 -> footprints:R0603
- R10, R11: value CR1/2WS-470K±5%-ST52 -> FRC0603F6340TS; footprint footprints:RES-TH_BD2.7-L6.2-P10.20-D0.4 -> footprints:R0603
- R12, R14, R20, R3, R5, R9: value CR1W-100K±5%-TT63 -> FRC0603F6340TS; footprint footprints:RES-TH_BD4.5-L11.0-P15.00-D0.7 -> footprints:R0603
- R13: value 820R 350V 500mW -> FRC0603F6340TS; footprint footprints:RES-TH_BD4.0-L10.5-P14.50-D0.6 -> footprints:R0603
- R16, R7: value CR1W-10M±5%-6T63 -> FRC0603F6340TS; footprint footprints:RES-TH_BD4.5-L11.0-P15.00-D0.7 -> footprints:R0603
- R17, R18, R2: value 1Meg 500V 250mW -> FRC0603F6340TS; footprint footprints:RES-TH_BD2.4-L6.3-P10.30-D0.6 -> footprints:R0603
- R19: value CF3WS-10KΩ±5%_T -> FRC0603F6340TS; footprint footprints:RES-TH_BD5.5-L15.0-P19.00-D0.8 -> footprints:R0603
- R21: value CR1/4W-47K±5%-ST52 -> CFR03SJ0153AA0_15k; footprint footprints:RES-TH_BD2.7-L6.2-P10.20-D0.4 -> footprints:RES-TH_BD6.0-L17.5-P21.50-D0.8
- R4, R8: value CR1/4W-2K7±5%-ST26 -> FRC0603F6340TS; footprint footprints:RES-TH_BD2.7-L6.2-P10.20-D0.4 -> footprints:R0603
- U1: value XSD366-094 -> IRM-03-5; footprint footprints:HEATSINK-TH_XSD366-094 -> footprints:PWRM-TH_IRM-03-5-DIP5
- U10: value 250pF 500V 5% -> KAQY214ATLD; footprint wb50_footprints:MICA_CAP_L15.5_W3.6_P8.7 -> footprints:SMD-4_L4.6-W6.4-P2.54-LS10.0-BR
- U11, U12, U13, U16, U9: value 500pF 500V 5% -> KAQY214ATLD; footprint wb50_footprints:MICA_CAP_L15.5_W3.6_P8.7 -> footprints:SMD-4_L4.6-W6.4-P2.54-LS10.0-BR
- U14, U15, U17, U25, U26: value 22n 630V 5% -> KAQY214ATLD; footprint wb50_footprints:MUSTARD_CAP_D8.5_L20.5_P25.5 -> footprints:SMD-4_L4.6-W6.4-P2.54-LS10.0-BR
- U18: value 470R 500V 2W -> KAQY214ATLD; footprint footprints:RES-TH_BD5.0-L15.5-P19.50-D0.7 -> footprints:SMD-4_L4.6-W6.4-P2.54-LS10.0-BR
- U19, U23: value 100n 630V 5% -> KAQY214ATLD; footprint wb50_footprints:MUSTARD_CAP_D10_L32_P40.4 -> footprints:SMD-4_L4.6-W6.4-P2.54-LS10.0-BR
- U2: value L7812CV-DG -> 16A 20mm 500V 5mm Plugin Fuse; footprint footprints:TO-220-3_L10.0-W4.5-P2.54-L -> footprints:FUSE-TH_L22.5-W10.8-P22.50_0031.8201.G
- U20: value CF2WS-82KΩ±5%_T -> KAQY214ATLD; footprint footprints:RES-TH_BD4.0-L11.5-P15.50-D0.7 -> footprints:SMD-4_L4.6-W6.4-P2.54-LS10.0-BR
- U21: value 100pF 500V 5% -> KAQY214ATLD; footprint wb50_footprints:MICA_CAP_L15.5_W3.6_P8.7 -> footprints:SMD-4_L4.6-W6.4-P2.54-LS10.0-BR
- U22, U27: value CR1/2W-220K±5%-XT52 -> KAQY214ATLD; footprint footprints:RES-TH_BD3.5-L9.0-P13.00-D0.5 -> footprints:SMD-4_L4.6-W6.4-P2.54-LS10.0-BR
- U24: value 4n7 630V 5% -> KAQY214ATLD; footprint wb50_footprints:MUSTARD_CAP_D8.5_L20.5_P25.5 -> footprints:SMD-4_L4.6-W6.4-P2.54-LS10.0-BR
- U3: value AB24S -> ESP32-ZERO; footprint footprints:ABS-SMD_L5.0-W4.4-P4.00-LS7.0-BL -> footprints:COMM-SMD_ESP32-ZERO
- U4: value CR1/2W-220K±5%-XT52 -> QNHC3; footprint footprints:RES-TH_BD3.5-L9.0-P13.00-D0.5 -> footprints:HALL-SENSOR_5P-P2.54-H13.5
- U5: value CR2W-68K±5%-9T73 -> 74HC595D,118; footprint footprints:RES-TH_BD5.0-L15.5-P19.50-D0.7 -> footprints:SOIC-16_L9.9-W3.9-P1.27-LS6.0-BL
- U6: value 500pF 500V 5% -> 74HC595D,118; footprint wb50_footprints:MICA_CAP_L15.5_W3.6_P8.7 -> footprints:SOIC-16_L9.9-W3.9-P1.27-LS6.0-BL
- U7: value 4n7 630V 5% -> 74HC595D,118; footprint wb50_footprints:MUSTARD_CAP_D8.5_L20.5_P25.5 -> footprints:SOIC-16_L9.9-W3.9-P1.27-LS6.0-BL
- U8: value 2n2 630V 5% -> KAQY214ATLD; footprint wb50_footprints:MUSTARD_CAP_D8.5_L20.5_P25.5 -> footprints:SMD-4_L4.6-W6.4-P2.54-LS10.0-BR
- moved U1 278.4 mm to (241.8, 92.5), turned to 180 degrees
- moved C3 276.4 mm to (233.0, 138.0), turned to -90 degrees
- moved D3 271.5 mm to (227.5, 179.0)
- moved U3 270.6 mm to (261.8, 118.0)
- moved U2 267.7 mm to (260.5, 72.5), turned to 0 degrees
- moved U19 257.7 mm to (257.0, 176.0), turned to 90 degrees
- moved C2 257.3 mm to (271.0, 103.0), turned to 0 degrees
- moved C4 250.8 mm to (254.5, 138.0), turned to -90 degrees
- moved C1 249.9 mm to (271.0, 106.0)
- moved D1 216.6 mm to (241.5, 112.0), turned to 180 degrees
- moved R21 186.0 mm to (226.2, 118.2), turned to -90 degrees
- moved U22 163.7 mm to (243.0, 176.0), turned to 90 degrees
- moved U7 151.7 mm to (267.0, 138.0), turned to 180 degrees
- moved U24 148.7 mm to (264.0, 158.0), turned to 90 degrees
- moved C5 140.1 mm to (273.5, 138.0), turned to -90 degrees
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Connections:
- C1 pad 1: +12V -> GND
- C1 pad 2: GND-AUX -> +5V
- C2 pad 1: Net-(U2-passive) -> GND
- C2 pad 2: GND-AUX -> +5V
- C3 pad 1: Net-(U2-passive) -> GND
- C3 pad 2: GND-AUX -> +5V
- C4 pad 1: +12V -> GND
- C4 pad 2: GND-AUX -> +5V
- C5 pad 1: Net-(V1A-C/K) -> GND
- C5 pad 2: GND-AUD -> +5V
- C6 pad 1: Net-(V1B-C/K) -> +325V
- C6 pad 2: GND-AUD -> GND-HV
- C7 pad 1: Net-(V2A-C/K) -> +182V
- C7 pad 2: GND-AUD -> GND-HV
- D1 pad 1: Net-(D1-K) -> AC1
- D1 pad 2: Net-(D1-A) -> AC2
- D3 pad 1: Net-(D3-K) -> +182V
- D4 pad 1: +12V -> Net-(D3-A)
- D4 pad 2: REL-SW -> GND-HV
- R1 pad 1: /Connectors/Audio_IN -> /NixieDigit1/Digital
- R1 pad 2: Net-(V1A-G) -> Net-(U10-A)
- R10 pad 1: /Pre Amp/PreAmp_OUT -> /NixieDigit10/Digital
- R10 pad 2: Net-(V2A-G) -> Net-(U17-A)
- R11 pad 1: Net-(V2A-G) -> /NixieDigit12/Digital
- R11 pad 2: GND-AUD -> Net-(U18-A)
- R12 pad 1: HV-D -> /NixieDigit13/Digital
- R12 pad 2: Net-(V2A-A/P) -> Net-(U19-A)
- R13 pad 1: Net-(V2A-C/K) -> /NixieDigit11/Digital
- R13 pad 2: GND-AUD -> Net-(U20-A)
- R14 pad 1: Net-(V2B-C/K) -> /NixieDigit14/Digital
- R14 pad 2: GND-AUD -> Net-(U21-A)
- R15 pad 1: Net-(V2B-C/K) -> /NixieDigit15/Digital
- R15 pad 2: Net-(R15-Pad2) -> Net-(U22-A)
- R16 pad 1: /Phase Inverter/PI_IN -> /NixieDigit16/Digital
- R16 pad 2: GND-AUD -> Net-(U23-A)
- R17 pad 1: Net-(V3A-G) -> /NixieDigit17/Digital
- R17 pad 2: Net-(R17-Pad2) -> Net-(U24-A)
- R18 pad 1: Net-(V3B-G) -> /NixieDigit18/Digital
- R18 pad 2: Net-(R17-Pad2) -> Net-(U25-A)
- R19 pad 1: Net-(R17-Pad2) -> /NixieDigit19/Digital
- R19 pad 2: Net-(R19-Pad2) -> Net-(U26-A)
- R2 pad 1: /Connectors/Audio_IN -> /NixieDigit2/Digital
- R2 pad 2: GND-AUD -> Net-(U8-A)
- R20 pad 1: HV-C -> /NixieDigit20/Digital
- R20 pad 2: Net-(V3B-A/P) -> Net-(U27-A)
- R21 pad 1: Net-(R19-Pad2) -> +325V
- R21 pad 2: Net-(R21-Pad2) -> +182V
- R3 pad 1: Net-(R3-Pad1) -> /NixieDigit3/Digital
- R3 pad 2: Net-(V1A-A/P) -> Net-(U9-A)
- R4 pad 1: Net-(V1A-C/K) -> /NixieDigit4/Digital
- R4 pad 2: GND-AUD -> Net-(U11-A)
- R5 pad 1: Net-(R5-Pad1) -> /NixieDigit5/Digital
- R5 pad 2: GND-AUD -> Net-(U12-A)
- R6 pad 1: Net-(R6-Pad1) -> /NixieDigit6/Digital
- R6 pad 2: Net-(V1B-G) -> Net-(U13-A)
- R7 pad 1: Net-(R6-Pad1) -> /NixieDigit7/Digital
- R7 pad 2: GND-AUD -> Net-(U14-A)
- R8 pad 1: Net-(V1B-C/K) -> /NixieDigit8/Digital
- R8 pad 2: GND-AUD -> Net-(U15-A)
- R9 pad 1: HV-E -> /NixieDigit9/Digital
- R9 pad 2: Net-(V1B-A/P) -> Net-(U16-A)
- U1 pad 1: unconnected-(U1-Pad1) -> AC1
- U10 pad 1: Net-(RV7-Pad3) -> Net-(U10-A)
- U10 pad 2: Net-(U10-Pad2) -> GND
- U11 pad 1: /Pre Amp/PreAmp_OUT -> Net-(U11-A)
- U11 pad 2: Net-(V2A-G) -> GND
- U12 pad 1: HV-D -> Net-(U12-A)
- U12 pad 2: Net-(V2A-A/P) -> GND
- U13 pad 1: Net-(V2B-C/K) -> Net-(U13-A)
- U13 pad 2: GND-AUD -> GND
- U14 pad 1: Net-(R15-Pad2) -> Net-(U14-A)
- U14 pad 2: Net-(RV2-Pad2) -> GND
- U15 pad 1: Net-(R15-Pad2) -> Net-(U15-A)
- U15 pad 2: Net-(RV3-Pad2) -> GND
- U16 pad 1: Net-(V2B-C/K) -> Net-(U16-A)
- U16 pad 2: Net-(RV4-Pad3) -> GND
- U17 pad 1: /Phase Inverter/PI_IN -> Net-(U17-A)
- U17 pad 2: Net-(V3A-G) -> GND
- U18 pad 1: Net-(V3A-C/K) -> Net-(U18-A)
- U18 pad 2: Net-(R17-Pad2) -> GND
- U19 pad 1: Net-(RV1-Pad2) -> Net-(U19-A)
- U19 pad 2: GND-AUD -> GND
- U2 pad 1: Net-(U2-passive) -> Net-(AC1-Pad1)
- U2 pad 2: GND-AUX -> AC1
- U20 pad 1: HV-C -> Net-(U20-A)
- U20 pad 2: Net-(V3A-A/P) -> GND
- U21 pad 1: Net-(V3A-A/P) -> Net-(U21-A)
- U21 pad 2: Net-(V3B-A/P) -> GND
- U22 pad 1: Net-(R21-Pad2) -> Net-(U22-A)
- U22 pad 2: /Connectors/NFB_IN -> GND
- U23 pad 1: Net-(V3B-G) -> Net-(U23-A)
- U23 pad 2: Net-(R19-Pad2) -> GND
- U24 pad 1: Net-(R21-Pad2) -> Net-(U24-A)
- U24 pad 2: /Connectors/NFB_IN -> GND
- U25 pad 1: Net-(V3A-A/P) -> Net-(U25-A)
- U25 pad 2: /Phase Inverter/PI_OUT_A -> GND
- U26 pad 1: Net-(V3B-A/P) -> Net-(U26-A)
- U26 pad 2: /Phase Inverter/PI_OUT_B -> GND
- U27 pad 1: /Phase Inverter/PI_OUT_A -> Net-(U27-A)
- U27 pad 2: /Power Amp/Bias-Set -> GND
- U3 pad 1: Net-(U2-passive) -> unconnected-(U3-USART0TX-Pad1)
- U3 pad 2: GND-AUX -> unconnected-(U3-USART0RX-Pad2)
- U3 pad 3: Net-(AC-IN5-Pad1) -> unconnected-(U3-GP13-Pad3)
- U3 pad 4: Net-(AC-IN4-Pad1) -> unconnected-(U3-GP12-Pad4)
- U4 pad 1: HV-E -> +5V
- U4 pad 2: Net-(R3-Pad1) -> GND
- U5 pad 1: Net-(U5-Pad1) -> /NixieDigit1/Digital
- U5 pad 2: Net-(R5-Pad1) -> /NixieDigit2/Digital
- U6 pad 1: Net-(R3-Pad1) -> /NixieDigit8/Digital
- U6 pad 2: Net-(V1A-A/P) -> /NixieDigit9/Digital
- U7 pad 1: Net-(V1A-A/P) -> /NixieDigit15/Digital
- U7 pad 2: Net-(U5-Pad1) -> /NixieDigit16/Digital
- U8 pad 1: Net-(V1B-A/P) -> Net-(U8-A)
- U8 pad 2: Net-(RV7-Pad3) -> GND
- U9 pad 1: Net-(RV7-Pad3) -> Net-(U9-A)
- U9 pad 2: Net-(U35-Pad1) -> GND
Routing:
- net GND-AUD: track 1221.7 -> 0.00 mm
- net +12V: track 817.0 -> 0.00 mm
- net GND-AUX: track 785.1 -> 0.00 mm, vias 1 -> 0
- net /Connectors/NFB_IN: track 262.8 -> 0.00 mm
- net Net-(Audo-From-FX1-Pad1): track 250.5 -> 0.00 mm
- net +5V: track 0.00 -> 250.4 mm, vias 0 -> 4
- net HV-B: track 234.7 -> 0.00 mm
- net Net-(RV2-Pad2): track 217.2 -> 0.00 mm
- net REL-SW: track 214.3 -> 0.00 mm
- net Net-(R19-Pad2): track 205.0 -> 0.00 mm, vias 1 -> 0
- net Net-(Audio-To-FX1-Pad1): track 201.4 -> 0.00 mm
- net Net-(RV7-Pad3): track 155.6 -> 0.00 mm
- net +182V: track 0.00 -> 146.7 mm, vias 0 -> 1
- net /Power Amp/Bias-Set: track 143.4 -> 0.00 mm
- net Net-(RV3-Pad2): track 141.0 -> 0.00 mm
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- added copper zone on B.Cu, net GND
- added copper zone on In2.Cu, net GND-HV
- removed copper zone on In2.Cu, net GND-AUD
- removed copper zone on In1.Cu, net GND-AUX
- removed copper zone on In2.Cu, net GND-PWR
Other:
- board size 405 x 190 mm -> 55 x 189 mm
- board text removed: "100k"
- board text removed: "100nF"
- board text removed: "10Meg"
- board text removed: "10k"
- board text removed: "10uF"
- board text removed: "12,6V~"
- board text removed: "15k"
- board text removed: "18uF"
- board text removed: "1Meg"
- board text removed: "1R"
- board text removed: "1k"
- board text removed: "1k5"
- board text removed: "220k"
- board text removed: "22n"
- board text removed: "22uF"
- board text removed: "250pF"
- board text removed: "2k7"
- board text removed: "2n2"
- board text removed: "33k"
- board text removed: "33uF"
- board text removed: "345V~"
- board text removed: "470R"
- board text removed: "470k"
- board text removed: "47R"
- board text removed: "47k"
- board text removed: "4k7"
- board text removed: "4n7"
- board text removed: "500pF"
- board text removed: "68k"
- board text removed: "820R"
- board text removed: "820nF"
- board text removed: "GND"
- board text removed: "Wechselbalg 50 V1.0 - Christopher Müller 10/25"

Commit message: update resistor, update voltages
Parts:
- added MH1: MountHole, MountingHole:MountingHole_3.2mm_M3, F.Cu at (351.0, 68.1)
- added MH2: MountHole, MountingHole:MountingHole_3.2mm_M3, F.Cu at (350.5, 193.0)
- added MH3: MountHole, MountingHole:MountingHole_3.2mm_M3, F.Cu at (294.0, 193.0)
- added MH4: MountHole, MountingHole:MountingHole_3.2mm_M3, F.Cu at (282.0, 193.0)
- added MH5: MountHole, MountingHole:MountingHole_3.2mm_M3, F.Cu at (224.5, 193.0)
- added MH6: MountHole, MountingHole:MountingHole_3.2mm_M3, F.Cu at (334.1, 150.2)
- added MH7: MountHole, MountingHole:MountingHole_3.2mm_M3, F.Cu at (299.9, 233.3)
- added R22: 0805W8F1202T5E, footprints:R0805, F.Cu at (226.4, 173.8)
- added R23: 0805W8F1202T5E, footprints:R0805, F.Cu at (231.9, 173.8)
- R1, R10, R11, R12, R13, R14, R15, R16, R17, R18, R19, R2, R20, R3, R4, R5, R6, R7, R8, R9: value FRC0603F6340TS -> 0603WAF2000T5E
- moved R16 158.8 mm to (139.8, 239.8), turned to 90 degrees
- moved U23 147.9 mm to (147.8, 239.8), turned to 180 degrees
- moved R13 138.9 mm to (139.5, 212.5), turned to 90 degrees
- moved R11 133.9 mm to (139.8, 218.0), turned to 90 degrees
- moved R17 130.9 mm to (139.2, 190.8), turned to 90 degrees
- moved R12 129.3 mm to (139.8, 223.5), turned to 90 degrees
- moved U20 128.8 mm to (147.5, 212.6), turned to 180 degrees
- moved R18 126.1 mm to (139.2, 196.2), turned to 90 degrees
- moved R14 125.5 mm to (139.8, 229.0), turned to 90 degrees
- moved U18 123.6 mm to (147.7, 218.0), turned to 180 degrees
- moved R15 122.5 mm to (139.8, 234.2), turned to 90 degrees
- moved R19 121.9 mm to (139.5, 201.8), turned to 90 degrees
- moved U24 121.3 mm to (147.2, 190.8), turned to 180 degrees
- moved U19 119.1 mm to (147.7, 223.4), turned to 180 degrees
- moved R20 118.1 mm to (139.5, 207.2), turned to 90 degrees
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Connections:
- C3 pad 2: +5V -> +3V3
- C4 pad 2: +5V -> +3V3
- C5 pad 2: +5V -> +3V3
- U3 pad 21: unconnected-(U3-3V3-Pad21) -> +3V3
- U5 pad 16: +5V -> +3V3
- U6 pad 16: +5V -> +3V3
- U7 pad 16: +5V -> +3V3
Routing:
- net /NixieDigit16/Digital: track 20.9 -> 324.8 mm, vias 2 -> 3
- net GND-HV: track 54.1 -> 336.6 mm, vias 20 -> 21
- net /NixieDigit19/Digital: track 37.7 -> 311.1 mm, vias 2 -> 5
- net /NixieDigit20/Digital: track 45.5 -> 308.5 mm, vias 2 -> 3
- net /NixieDigit15/Digital: track 61.6 -> 323.1 mm, vias 2 -> 3
- net /NixieDigit17/Digital: track 26.6 -> 273.6 mm, vias 2 -> 5
- net /NixieDigit18/Digital: track 30.3 -> 274.5 mm, vias 2 -> 5
- net /NixieDigit9/Digital: track 51.2 -> 291.3 mm, vias 0 -> 5
- net /NixieDigit14/Digital: track 39.7 -> 277.7 mm, vias 1 -> 6
- net /NixieDigit13/Digital: track 40.8 -> 276.1 mm, vias 1 -> 5
- net /NixieDigit12/Digital: track 44.4 -> 276.6 mm, vias 1 -> 5
- net /NixieDigit8/Digital: track 67.5 -> 294.3 mm, vias 0 -> 5
- net /NixieDigit11/Digital: track 54.6 -> 278.9 mm, vias 0 -> 5
- net /NixieDigit10/Digital: track 59.1 -> 257.2 mm, vias 0 -> 6
- net /NixieDigit4/Digital: track 78.7 -> 259.2 mm, vias 1 -> 4
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- added copper zone on F.Cu, net +182V
- added copper zone on F.Cu, net GND
- added copper zone on In2.Cu, net GND
- added copper zone on In1.Cu, net GND-HV
- removed copper zone on B.Cu, net GND
- removed copper zone on In2.Cu, net GND-HV
Other:
- board size 55 x 189 mm -> 241.7 x 190 mm
- board text added: "Nixie Addon Board V1.0 - 10/2025 - Christopher Müller"
- board text added: "W"
- board text added: "echselbalg 50"

Commit message: update schmatic
Parts:
- added C8: 0603B472K500NT, footprints:C0603, F.Cu at (330.8, 81.7)
- added R24: 0603WAF1201T5E, footprints:R0603, F.Cu at (337.5, 79.0)
- added R25: 0603WAF3301T5E, footprints:R0603, F.Cu at (330.8, 79.0)
- R22, R23: value 0805W8F1202T5E -> 0603WAF1002T5E; footprint footprints:R0805 -> footprints:R0603
- moved MH5 4.00 mm to (228.5, 193.0)
- moved MH4 3.50 mm to (278.5, 193.0)
- moved MH2 3.25 mm to (347.2, 193.0)
- moved MH3 3.25 mm to (297.2, 193.0)
- moved C6 2.34 mm to (323.0, 108.4)
- moved R22 0.30 mm to (226.4, 174.1)
- moved R23 0.11 mm to (231.8, 173.9)
Connections:
- NX1 pad 11: +182V -> /Anode1
- NX2 pad 11: +182V -> /Anode2
- U3 pad 15: unconnected-(U3-GP6-Pad15) -> Net-(U3-GP6)
- U3 pad 18: Net-(U3-GP3) -> unconnected-(U3-GP3-Pad18)
- U4 pad 3: Net-(U3-GP3) -> Net-(U4-OUT)
Routing:
- net +182V: track 288.8 -> 147.8 mm, vias 3 -> 1
- net /Anode2: track 0.00 -> 79.6 mm, vias 0 -> 1
- net /Anode1: track 0.00 -> 62.0 mm, vias 0 -> 1
- net Net-(U3-GP6): track 0.00 -> 10.5 mm
- net +3V3: track 133.8 -> 142.0 mm
- net Net-(U3-GP3): track 6.71 -> 0.00 mm
- net Net-(U4-OUT): track 0.00 -> 6.00 mm
- net /NixieDigit1/Digital: track 237.7 -> 240.7 mm
- net /NixieDigit14/Digital: track 277.7 -> 280.6 mm
- net /NixieDigit13/Digital: track 276.1 -> 278.9 mm
- net /NixieDigit12/Digital: track 276.6 -> 279.3 mm
- net +5V: track 109.8 -> 112.4 mm
- net /NixieDigit20/Digital: track 308.5 -> 311.1 mm
- net +325V: track 23.3 -> 25.9 mm
- net /NixieDigit19/Digital: track 311.1 -> 312.7 mm
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- added copper zone on F.Cu, net /Anode1
- added copper zone on F.Cu, net /Anode2
- removed copper zone on F.Cu, net +182V
Other:
- outline, holes or cut-outs redrawn

Commit message: fix: schematic mistakes corrected
Routing:
- net GND: vias 32 -> 34
- added copper zone on In1.Cu, net GND
Other:
- board text added: "Nixie Addon Board V1.1 - 10/2025 - Christopher Müller"
- board text removed: "Nixie Addon Board V1.0 - 10/2025 - Christopher Müller"
Changed lines of the file:
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@@
 		)
 	)
-	(gr_text "Nixie Addon Board V1.0 - 10/2025 - Christopher Müller"
+	(gr_text "Nixie Addon Board V1.1 - 10/2025 - Christopher Müller"
 		(at 219.15 154.63 0)
 		(layer "F.SilkS")
@@
 	)
 	(via
+		(at 353.5 79)
+		(size 1)
+		(drill 0.5)
+		(layers "F.Cu" "B.Cu")
+		(free yes)
+		(net 4)
+	)
+	(via
 		(at 301.5 96.5)
 		(size 1)
@@
 	)
 	(via
+		(at 352 79)
+		(size 1)
+		(drill 0.5)
+		(layers "F.Cu" "B.Cu")
+		(free yes)
+		(net 4)
+	)
+	(via
 		(at 330.65 95.392857)
 		(size 1)
@@
 		(polygon
 			(pts
-				(xy 278 86) (xy 278 97.75) (xy 308 97.75) (xy 308 86)
+				(xy 278 84) (xy 278 98.75) (xy 308 98.75) (xy 308 84)
 			)
 		)
@@
 	)
 	(zone
+		(net 4)
+		(net_name "GND")
+		(layer "In1.Cu")
+		(hatch edge 0.5)
+		(priority 5)
+		(connect_pads
+			(clearance 0.5)
+		)
+		(min_thickness 0.25)
+		(filled_areas_thickness no)
+		(fill yes
+			(thermal_gap 0.5)
+			(thermal_bridge_width 0.5)
+		)
+		(polygon
+			(pts
+				(xy 332 98.5) (xy 327 98.5) (xy 327 77.5) (xy 354.5 77.5) (xy 354.5 84) (xy 332 84)
+			)
+		)
+	)
+	(zone
 		(net 5)
 		(net_name "GND-HV")
@@
 		(polygon
 			(pts
-				(xy 278 86) (xy 278 97.75) (xy 333.25 97.75) (xy 333 86)
+				(xy 278 84) (xy 278 98.75) (xy 333.25 98.75) (xy 333 84)
 			)
 		)
